Commit message: urdf学习

File: chapt6/chapt6_ws/src/fishbot_description/urdf/first_robot.urdf (robot description, URDF)
Before this commit: robot robot_name, 1 links, 0 joints
Links:
- added link imu_link; visual box size=0.02 0.02 0.02
Joints:
- added joint imu_joint: type fixed, parent base_link, child imu_link, origin xyz=0.0 0.0 0.1 rpy=0.0 0.0 0.0
