Commit message: 完成fishbot个运动部件和传感器的建模

File: chapt6/chapt6_ws/install/fishbot_description/share/fishbot_description/urdf/first_robot.xacro (robot description, xacro)
@@ -44,5 +44,5 @@
             <child link="${imu_name}_link"/>
             <!-- 关节的原点位置和姿态-->
-            <origin xyz="0.0 0.0 0.1" rpy="0.0 0.0 0.0"/>
+            <origin xyz="0.0 0.0 0.0" rpy="0.0 0.0 0.0"/>
         </joint>
     </xacro:macro>
